Commit message: moveit_controllers corrections rotate the gripper in urdf

File: lbr_description/urdf/iiwa14_2f85/iiwa14_2f85.xacro (robot description, xacro)
@@ -23,4 +23,5 @@
         system_config_path="$(arg system_config_path)" />
     <!-- gripper -->
+    <!-- SHOULD PASS robot_name AS PARAMETER/ARGUMENT -->
     <xacro:include filename="$(find lbr_description)/urdf/iiwa14_2f85/robotiq_2f_85_gripper.urdf.xacro" />
 </robot>

File: lbr_description/urdf/iiwa14_2f85/robotiq_2f_85_gripper.urdf.xacro (robot description, xacro)
@@ -3,4 +3,5 @@
     <!-- parameters -->
     <xacro:arg name="use_fake_hardware" default="true" />
+    <xacro:arg name="robot_name" default="lbr" />
     <!-- Import macros -->
     <xacro:include filename="$(find lbr_description)/urdf/iiwa14_2f85/robotiq_2f_85_macro.urdf.xacro" />
@@ -8,6 +9,6 @@
     <link name="world" />
     -->
-    <xacro:robotiq_gripper name="RobotiqGripperHardwareInterface" prefix="" parent="lbr_link_ee" use_fake_hardware="$(arg use_fake_hardware)">
-        <origin xyz="0 0 0" rpy="0 0 0" />
+    <xacro:robotiq_gripper name="RobotiqGripperHardwareInterface" prefix="" parent="$(arg robot_name)_link_ee" use_fake_hardware="$(arg use_fake_hardware)">
+        <origin xyz="0 0 0.0143" rpy="0 0 90" />
     </xacro:robotiq_gripper>
 </robot>
