Commit message: change gripper to proper end effector

File: lbr_description/urdf/iiwa14_2f85/robotiq_2f_85_gripper.urdf.xacro (robot description, xacro)
@@ -3,5 +3,4 @@
     <!-- parameters -->
     <xacro:arg name="use_fake_hardware" default="true" />
-    <xacro:arg name="robot_name" default="lbr" />
     <!-- Import macros -->
     <xacro:include filename="$(find lbr_description)/urdf/iiwa14_2f85/robotiq_2f_85_macro.urdf.xacro" />
@@ -9,6 +8,6 @@
     <link name="world" />
     -->
-    <xacro:robotiq_gripper name="RobotiqGripperHardwareInterface" prefix="" parent="$(arg robot_name)_link_ee" use_fake_hardware="$(arg use_fake_hardware)">
-        <origin xyz="0 0 0.0143" rpy="0 0 90" />
+    <xacro:robotiq_gripper name="RobotiqGripperHardwareInterface" prefix="" parent="lbr_link_ee" use_fake_hardware="$(arg use_fake_hardware)">
+        <origin xyz="0 0 0" rpy="0 0 1.5708" />
     </xacro:robotiq_gripper>
 </robot>
