Commit message: ajout dummy_link_ee pour simuler le gripper

File: lbr_description/urdf/iiwa14_2f85/iiwa14_2f85_description.xacro (robot description, xacro)
@@ -270,5 +270,12 @@
             <origin xyz="0 0 0.035" rpy="0 0 0" />
         </joint>
+        <joint name="${robot_name}_joint_dummy_ee" type="fixed">
+            <parent link="${robot_name}_link_7" />
+            <child link="${robot_name}_link_dummy_ee" />
+            <origin xyz="0 0 0.135" rpy="0 0 0" />
+        </joint>
         <link name="${robot_name}_link_ee">
+        </link>
+        <link name="${robot_name}_link_dummy_ee">
         </link>
     </xacro:macro>

File: lbr_description/urdf/iiwa14_2f85/robotiq_2f_85_macro.urdf.xacro (robot description, xacro)
@@ -275,4 +275,12 @@
             <mimic joint="${prefix}robotiq_85_left_knuckle_joint" />
         </joint>
+        <joint name="${prefix}robotiq_85_tcp_joint" type="fixed">
+            <parent link="${prefix}robotiq_85_base_link" />
+            <child link="${prefix}robotiq_85_tcp_link" />
+            <axis xyz="0 -1 0" />
+            <origin xyz="0 0 0.135" rpy="0 0 0" />
+        </joint>
+        <link name="${prefix}robotiq_85_tcp_link">
+        </link>
     </xacro:macro>
 </robot>
